Commit message: Se han recogido los parametros en un archivo

File: src/ow_robot/description/robot.gazebo.xacro (robot description, xacro)
@@ -44,12 +44,11 @@
     </gazebo>
     <gazebo>
-        <plugin name="object_controller" filename="libgazebo_ros_planar_move.so">
+        <plugin name="omni_steering" filename="libgazebo_ros_planar_move.so">
         <commandTopic>cmd_vel</commandTopic>
         <odometryTopic>odom</odometryTopic>
         <odometryFrame>odom</odometryFrame>
-        <odometryRate>20.0</odometryRate>
+        <odometryRate>100.0</odometryRate>
         <robotBaseFram>base_footprint</robotBaseFram>
-        <publish_odom>true</publish_odom>
-        <publish_odom_tf>true</publish_odom_tf>
+        <publishTF>True</publishTF>
         </plugin>
   </gazebo>

File: src/ow_robot/description/robot_core.xacro (robot description, xacro)
@@ -2,16 +2,5 @@
 <robot xmlns:xacro="http://www.ros.org/wiki/xacro" >
     <xacro:include filename="inertial_macros.xacro"/>
-    <xacro:property name="altura_eje_base" value="0.02335"/>
-    <xacro:property name="grosor_base" value="0.006"/>
-    <xacro:property name="radio_rueda" value="0.05"/>
-    <xacro:property name="grosor_robot" value="0.08375"/>
-    <xacro:property name="offset_perfiles" value="0.1205"/>
-    <xacro:property name="grosor_perfiles" value="0.02"/>
-    <xacro:property name="largo_perfiles" value="0.25"/>
-    <xacro:property name="offset_esquinas" value="0.19"/>
-    <xacro:property name="ancho_servo" value="0.05715"/>
-    <xacro:property name="largo_servo" value="0.10985"/>
-    <xacro:property name="offset_vertical_servo" value="0.0045"/>
-    <xacro:property name="offset_horizontal_servo" value="0.004"/>
+    <xacro:include filename="params.xacro"/>
     <!--Materiales para visualizacion en RVIZ-->
     <xacro:include filename="materials.xacro"/>
@@ -19,5 +8,12 @@
     <xacro:include filename="robot.gazebo.xacro"/>
     <!-- BASE LINK -->
+    <!-- root link, on the ground just below the model origin -->
     <link name="base_footprint">
+    <visual>
+        <origin xyz="0 0 0" rpy="0 0 0" />
+        <geometry>
+            <box size="0.001 0.001 0.001" />
+        </geometry>
+        </visual>
     </link>
     <!-- PLACA INFERIOR -->
