Commit message: Se ha creado el nodo que calcula la cinematica inversa

File: src/ow_robot/description/robot_core.xacro (robot description, xacro)
@@ -290,5 +290,5 @@
             <origin xyz="0 0 0"/>
             <geometry>
-                <mesh filename="file://$(find ow_robot)/meshes/esquina.stl" scale="0.001 0.001 0.001"/>
+                <mesh filename="file://$(find ow_robot)/meshes/esquina.dae" scale="0.001 0.001 0.001"/>
             </geometry>
             <material name="blue"/>
@@ -388,5 +388,5 @@
         <parent link="servo_front"/>
         <child link="rueda_front"/>
-        <origin xyz="${ancho_servo/2} 0.026575 0.15 " rpy="0 0 0"/>
+        <origin xyz="${ancho_servo/2} 0.026575 0.15 " rpy="${pi/2} 0 0"/>
         <axis xyz="0 0 1"/>
     </joint>
@@ -395,5 +395,5 @@
             <origin xyz="0 0 0"/>
             <geometry>
-               <cylinder radius="0.050" length="0.04"/>
+               <mesh filename="file://$(find ow_robot)/meshes/esquina.dae" scale="0.001 0.001 0.001"/>
             </geometry>
             <material name="black"/>
